File: materiel/carte-v1/kicad/alimentation.kicad_sch (KiCad schematic)
At the start: 33 parts, among them U4 BQ25180YBGR, U5 TPS63900DSKR, U6 TPS22965DSGR, U7 MAX17048G+T10

Commit message: fix(materiel): revue complète de la carte V1 avant commande
- microcontrôleur STM32U585CIT6 à la place du STM32U575CIT6, en rupture chez JLCPCB (même brochage, ADR 0042 point 11)
- VBIAS de U6 prise sur la batterie et couloir réservé à la commande du modem : la broche ON n'était plus routable sous le bord du module
- cuivre interne de 1 oz (empilement JLC061211-3313) : chemin du modem à 20 mΩ au lieu de 33 mΩ ; lignes d'antenne à 0,186 mm pour rester à 50 Ω
- placement à la convention JLCPCB (face inférieure à 180° moins l'angle KiCad), empreintes comparées à LCSC, nomenclature par référence LCSC
- hauteurs de la face inférieure d'après les fiches des fabricants (1,35 mm), modèles 3D relatifs au projet, L1 ramenée à 1,2 mm
- finition : vias thermiques en double et cuivre mort retirés ; vias de plan : perçages du même réseau, îlots, via dans la pastille en dégageant le routage
- fiche de commande complète, guide PDF de commande et de mise en service, cahier § 6 tranché
Parts:
- C3: value 1 µF -> 4,7 µF; Fabricant CL05A105KA5NQNC -> CL05A475MP5NRNC; LCSC C52923 -> C23733; Note (none) -> BAT : au moins 1 µF effectif sous 4,2 V (fiche TI) ; un 1 µ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
Connections:
- net VBAT: now also U6.4 (VBIAS)
- net VBAT_MES: no longer U6.4 (VBIAS)
Changed lines of the file:
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@@
 (global_label "VSYS" (shape passive) (at 334.01 44.45 90) (fields_autoplaced yes) (effects (font (size 1.27 1.27)) (justify left)) (property "Intersheetrefs" "${INTERSHEET_REFS}" (at 334.01 44.45 0) (effects (font (size 1.27 1.27)) (hide yes))))
 (global_label "GND" (shape passive) (at 334.01 52.07 270) (fields_autoplaced yes) (effects (font (size 1.27 1.27)) (justify right)) (property "Intersheetrefs" "${INTERSHEET_REFS}" (at 334.01 52.07 0) (effects (font (size 1.27 1.27)) (hide yes))))
-(symbol (lib_id "Device:C") (at 369.57 48.26 0) (unit 1) (exclude_from_sim no) (in_bom yes) (on_board yes) (dnp no) (property "Reference" "C3" (at 369.57 44.26 0) (effects (font (size 1.27 1.27)))) (property "Value" "1 µF" (at 369.57 42.26 0) (effects (font (size 1.27 1.27)))) (property "Footprint" "Capacitor_SMD:C_0402_1005Metric" (at 369.57 48.26 0) (effects (font (size 1.27 1.27)) (hide yes))) (property "Datasheet" "" (at 369.57 48.26 0) (effects (font (size 1.27 1.27)) (hide yes))) (property "Fabricant" "CL05A105KA5NQNC" (at 369.57 48.26 0) (effects (font (size 1.27 1.27)) (hide yes))) (property "LCSC" "C52923" (at 369.57 48.26 0) (effects (font (size 1.27 1.27)) (hide yes))) (property "Note" "" (at 369.57 48.26 0) (effects (font (size 1.27 1.27)) (hide yes))) (pin "1") (pin "2") (instances (project "fasoguardian-v1" (path "/575af4e1-e15c-5e7c-a7b6-b5580dce1053/06663894-3f9d-535a-8063-8860181f393f" (reference "C3") (unit 1)))))
+(symbol (lib_id "Device:C") (at 369.57 48.26 0) (unit 1) (exclude_from_sim no) (in_bom yes) (on_board yes) (dnp no) (property "Reference" "C3" (at 369.57 44.26 0) (effects (font (size 1.27 1.27)))) (property "Value" "4,7 µF" (at 369.57 42.26 0) (effects (font (size 1.27 1.27)))) (property "Footprint" "Capacitor_SMD:C_0402_1005Metric" (at 369.57 48.26 0) (effects (font (size 1.27 1.27)) (hide yes))) (property "Datasheet" "" (at 369.57 48.26 0) (effects (font (size 1.27 1.27)) (hide yes))) (property "Fabricant" "CL05A475MP5NRNC" (at 369.57 48.26 0) (effects (font (size 1.27 1.27)) (hide yes))) (property "LCSC" "C23733" (at 369.57 48.26 0) (effects (font (size 1.27 1.27)) (hide yes))) (property "Note" "BAT : au moins 1 µF effectif sous 4,2 V (fiche TI) ; un 1 µF 0402 en perd 20 %" (at 369.57 48.26 0) (effects (font (size 1.27 1.27)) (hide yes))) (pin "1") (pin "2") (instances (project "fasoguardian-v1" (path "/575af4e1-e15c-5e7c-a7b6-b5580dce1053/06663894-3f9d-535a-8063-8860181f393f" (reference "C3") (unit 1)))))
 (global_label "VBAT" (shape passive) (at 369.57 44.45 90) (fields_autoplaced yes) (effects (font (size 1.27 1.27)) (justify left)) (property "Intersheetrefs" "${INTERSHEET_REFS}" (at 369.57 44.45 0) (effects (font (size 1.27 1.27)) (hide yes))))
 (global_label "GND" (shape passive) (at 369.57 52.07 270) (fields_autoplaced yes) (effects (font (size 1.27 1.27)) (justify right)) (property "Intersheetrefs" "${INTERSHEET_REFS}" (at 369.57 52.07 0) (effects (font (size 1.27 1.27)) (hide yes))))
@@
 (global_label "VBAT_MES" (shape passive) (at 115.57000000000001 105.41 180) (fields_autoplaced yes) (effects (font (size 1.27 1.27)) (justify right)) (property "Intersheetrefs" "${INTERSHEET_REFS}" (at 115.57000000000001 105.41 0) (effects (font (size 1.27 1.27)) (hide yes))))
 (global_label "MODEM_EN" (shape passive) (at 115.57000000000001 107.95 180) (fields_autoplaced yes) (effects (font (size 1.27 1.27)) (justify right)) (property "Intersheetrefs" "${INTERSHEET_REFS}" (at 115.57000000000001 107.95 0) (effects (font (size 1.27 1.27)) (hide yes))))
-(global_label "VBAT_MES" (shape passive) (at 115.57000000000001 110.49 180) (fields_autoplaced yes) (effects (font (size 1.27 1.27)) (justify right)) (property "Intersheetrefs" "${INTERSHEET_REFS}" (at 115.57000000000001 110.49 0) (effects (font (size 1.27 1.27)) (hide yes))))
+(global_label "VBAT" (shape passive) (at 115.57000000000001 110.49 180) (fields_autoplaced yes) (effects (font (size 1.27 1.27)) (justify right)) (property "Intersheetrefs" "${INTERSHEET_REFS}" (at 115.57000000000001 110.49 0) (effects (font (size 1.27 1.27)) (hide yes))))
 (global_label "GND" (shape passive) (at 140.97 110.49 0) (fields_autoplaced yes) (effects (font (size 1.27 1.27)) (justify left)) (property "Intersheetrefs" "${INTERSHEET_REFS}" (at 140.97 110.49 0) (effects (font (size 1.27 1.27)) (hide yes))))
 (global_label "MODEM_CT" (shape passive) (at 140.97 107.95 0) (fields_autoplaced yes) (effects (font (size 1.27 1.27)) (justify left)) (property "Intersheetrefs" "${INTERSHEET_REFS}" (at 140.97 107.95 0) (effects (font (size 1.27 1.27)) (hide yes))))
