File: materiel/carte-v1/kicad/fasoguardian-v1.kicad_sch (KiCad schematic)
At the start: 0 parts

Commit message: fix(materiel): revue complète de la carte V1 avant commande
- microcontrôleur STM32U585CIT6 à la place du STM32U575CIT6, en rupture chez JLCPCB (même brochage, ADR 0042 point 11)
- VBIAS de U6 prise sur la batterie et couloir réservé à la commande du modem : la broche ON n'était plus routable sous le bord du module
- cuivre interne de 1 oz (empilement JLC061211-3313) : chemin du modem à 20 mΩ au lieu de 33 mΩ ; lignes d'antenne à 0,186 mm pour rester à 50 Ω
- placement à la convention JLCPCB (face inférieure à 180° moins l'angle KiCad), empreintes comparées à LCSC, nomenclature par référence LCSC
- hauteurs de la face inférieure d'après les fiches des fabricants (1,35 mm), modèles 3D relatifs au projet, L1 ramenée à 1,2 mm
- finition : vias thermiques en double et cuivre mort retirés ; vias de plan : perçages du même réseau, îlots, via dans la pastille en dégageant le routage
- fiche de commande complète, guide PDF de commande et de mise en service, cahier § 6 tranché
Other:
- sheet Microcontrôleur STM32U575 renamed Microcontrôleur STM32U585
Changed lines of the file:
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@@
 (sheet (at 210 40) (size 70 40) (exclude_from_sim no) (in_bom yes) (on_board yes) (dnp no) (fields_autoplaced yes) (stroke (width 0.1524) (type solid)) (fill (color 0 0 0 0.0000)) (property "Sheetname" "Antennes LTE et GNSS" (at 210 39 0) (effects (font (size 1.27 1.27)) (justify left bottom))) (property "Sheetfile" "radio.kicad_sch" (at 210 81 0) (effects (font (size 1.27 1.27)) (justify left top))) (instances (project "fasoguardian-v1" (path "/575af4e1-e15c-5e7c-a7b6-b5580dce1053" (page "4")))))
 (sheet (at 300 40) (size 70 40) (exclude_from_sim no) (in_bom yes) (on_board yes) (dnp no) (fields_autoplaced yes) (stroke (width 0.1524) (type solid)) (fill (color 0 0 0 0.0000)) (property "Sheetname" "Carte SIM" (at 300 39 0) (effects (font (size 1.27 1.27)) (justify left bottom))) (property "Sheetfile" "sim.kicad_sch" (at 300 81 0) (effects (font (size 1.27 1.27)) (justify left top))) (instances (project "fasoguardian-v1" (path "/575af4e1-e15c-5e7c-a7b6-b5580dce1053" (page "5")))))
-(sheet (at 30 100) (size 70 40) (exclude_from_sim no) (in_bom yes) (on_board yes) (dnp no) (fields_autoplaced yes) (stroke (width 0.1524) (type solid)) (fill (color 0 0 0 0.0000)) (property "Sheetname" "Microcontrôleur STM32U575" (at 30 99 0) (effects (font (size 1.27 1.27)) (justify left bottom))) (property "Sheetfile" "microcontroleur.kicad_sch" (at 30 141 0) (effects (font (size 1.27 1.27)) (justify left top))) (instances (project "fasoguardian-v1" (path "/575af4e1-e15c-5e7c-a7b6-b5580dce1053" (page "6")))))
+(sheet (at 30 100) (size 70 40) (exclude_from_sim no) (in_bom yes) (on_board yes) (dnp no) (fields_autoplaced yes) (stroke (width 0.1524) (type solid)) (fill (color 0 0 0 0.0000)) (property "Sheetname" "Microcontrôleur STM32U585" (at 30 99 0) (effects (font (size 1.27 1.27)) (justify left bottom))) (property "Sheetfile" "microcontroleur.kicad_sch" (at 30 141 0) (effects (font (size 1.27 1.27)) (justify left top))) (instances (project "fasoguardian-v1" (path "/575af4e1-e15c-5e7c-a7b6-b5580dce1053" (page "6")))))
 (sheet (at 120 100) (size 70 40) (exclude_from_sim no) (in_bom yes) (on_board yes) (dnp no) (fields_autoplaced yes) (stroke (width 0.1524) (type solid)) (fill (color 0 0 0 0.0000)) (property "Sheetname" "Capteurs, élément sécurisé et mémoire" (at 120 99 0) (effects (font (size 1.27 1.27)) (justify left bottom))) (property "Sheetfile" "capteurs.kicad_sch" (at 120 141 0) (effects (font (size 1.27 1.27)) (justify left top))) (instances (project "fasoguardian-v1" (path "/575af4e1-e15c-5e7c-a7b6-b5580dce1053" (page "7")))))
 (sheet (at 210 100) (size 70 40) (exclude_from_sim no) (in_bom yes) (on_board yes) (dnp no) (fields_autoplaced yes) (stroke (width 0.1524) (type solid)) (fill (color 0 0 0 0.0000)) (property "Sheetname" "Translateurs 1,8 V / 3,3 V" (at 210 99 0) (effects (font (size 1.27 1.27)) (justify left bottom))) (property "Sheetfile" "niveaux.kicad_sch" (at 210 141 0) (effects (font (size 1.27 1.27)) (justify left top))) (instances (project "fasoguardian-v1" (path "/575af4e1-e15c-5e7c-a7b6-b5580dce1053" (page "8")))))
