File: materiel/carte-v1/kicad/microcontroleur.kicad_sch (KiCad schematic)
At the start: 22 parts, among them J7 SWD Tag-Connect, U1 STM32U575CIT6, Y1 32,768 kHz

Commit message: fix(materiel): revue complète de la carte V1 avant commande
- microcontrôleur STM32U585CIT6 à la place du STM32U575CIT6, en rupture chez JLCPCB (même brochage, ADR 0042 point 11)
- VBIAS de U6 prise sur la batterie et couloir réservé à la commande du modem : la broche ON n'était plus routable sous le bord du module
- cuivre interne de 1 oz (empilement JLC061211-3313) : chemin du modem à 20 mΩ au lieu de 33 mΩ ; lignes d'antenne à 0,186 mm pour rester à 50 Ω
- placement à la convention JLCPCB (face inférieure à 180° moins l'angle KiCad), empreintes comparées à LCSC, nomenclature par référence LCSC
- hauteurs de la face inférieure d'après les fiches des fabricants (1,35 mm), modèles 3D relatifs au projet, L1 ramenée à 1,2 mm
- finition : vias thermiques en double et cuivre mort retirés ; vias de plan : perçages du même réseau, îlots, via dans la pastille en dégageant le routage
- fiche de commande complète, guide PDF de commande et de mise en service, cahier § 6 tranché
Parts:
- U1: value STM32U575CIT6 -> STM32U585CIT6; symbol MCU_ST_STM32U5:STM32U575CITx -> MCU_ST_STM32U5:STM32U585CITx; Fabricant STM32U575CIT6 -> STM32U585CIT6; LCSC C5271014 -> C5271027; Note (none) -> STM32U575 et accélérateurs cryptographiques (AES, PKA, HASH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
Other:
- title: Microcontrôleur STM32U575 -> Microcontrôleur STM32U585
Changed lines of the file:
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@@
 (kicad_sch (version 20250114) (generator "eeschema") (generator_version "9.0")
  (paper "A3")
-(title_block (title "Microcontrôleur STM32U575") (date "2026-10-22") (rev "V1.0") (company "Collectif Dedsec — FasoGuardian") (comment 1 "Bracelet FasoGuardian, carte V1 (FG-DOC-08 § 12)") (comment 2 "Généré par materiel/carte-v1/conception/generer_schema.py depuis carte.py"))
-(symbol (lib_id "MCU_ST_STM32U5:STM32U575CITx") (at 59.69 85.09 0) (unit 1) (exclude_from_sim no) (in_bom yes) (on_board yes) (dnp no) (property "Reference" "U1" (at 59.69 81.09 0) (effects (font (size 1.27 1.27)))) (property "Value" "STM32U575CIT6" (at 59.69 79.09 0) (effects (font (size 1.27 1.27)))) (property "Footprint" "Package_QFP:LQFP-48_7x7mm_P0.5mm" (at 59.69 85.09 0) (effects (font (size 1.27 1.27)) (hide yes))) (property "Datasheet" "" (at 59.69 85.09 0) (effects (font (size 1.27 1.27)) (hide yes))) (property "Fabricant" "STM32U575CIT6" (at 59.69 85.09 0) (effects (font (size 1.27 1.27)) (hide yes))) (property "LCSC" "C5271014" (at 59.69 85.09 0) (effects (font (size 1.27 1.27)) (hide yes))) (property "Note" "" (at 59.69 85.09 0) (effects (font (size 1.27 1.27)) (hide yes))) (pin "1") (pin "2") (pin "3") (pin "4") (pin "5") (pin "6") (pin "7") (pin "8") (pin "9") (pin "10") (pin "11") (pin "12") (pin "13") (pin "14") (pin "15") (pin "16") (pin "17") (pin "18") (pin "19") (pin "20") (pin "21") (pin "22") (pin "23") (pin "24") (pin "25") (pin "26") (pin "27") (pin "28") (pin "29") (pin "30") (pin "31") (pin "32") (pin "33") (pin "34") (pin "35") (pin "36") (pin "37") (pin "38") (pin "39") (pin "40") (pin "41") (pin "42") (pin "43") (pin "44") (pin "45") (pin "46") (pin "47") (pin "48") (instances (project "fasoguardian-v1" (path "/575af4e1-e15c-5e7c-a7b6-b5580dce1053/f00164bc-1320-5990-b001-d3d612522a42" (reference "U1") (unit 1)))))
+(title_block (title "Microcontrôleur STM32U585") (date "2026-10-22") (rev "V1.0") (company "Collectif Dedsec — FasoGuardian") (comment 1 "Bracelet FasoGuardian, carte V1 (FG-DOC-08 § 12)") (comment 2 "Généré par materiel/carte-v1/conception/generer_schema.py depuis carte.py"))
+(symbol (lib_id "MCU_ST_STM32U5:STM32U585CITx") (at 59.69 85.09 0) (unit 1) (exclude_from_sim no) (in_bom yes) (on_board yes) (dnp no) (property "Reference" "U1" (at 59.69 81.09 0) (effects (font (size 1.27 1.27)))) (property "Value" "STM32U585CIT6" (at 59.69 79.09 0) (effects (font (size 1.27 1.27)))) (property "Footprint" "Package_QFP:LQFP-48_7x7mm_P0.5mm" (at 59.69 85.09 0) (effects (font (size 1.27 1.27)) (hide yes))) (property "Datasheet" "" (at 59.69 85.09 0) (effects (font (size 1.27 1.27)) (hide yes))) (property "Fabricant" "STM32U585CIT6" (at 59.69 85.09 0) (effects (font (size 1.27 1.27)) (hide yes))) (property "LCSC" "C5271027" (at 59.69 85.09 0) (effects (font (size 1.27 1.27)) (hide yes))) (property "Note" "STM32U575 et accélérateurs cryptographiques (AES, PKA, HASH), même brochage : le U575CIT6 est en rupture chez JLCPCB (ADR 0042, point 11)" (at 59.69 85.09 0) (effects (font (size 1.27 1.27)) (hide yes))) (pin "1") (pin "2") (pin "3") (pin "4") (pin "5") (pin "6") (pin "7") (pin "8") (pin "9") (pin "10") (pin "11") (pin "12") (pin "13") (pin "14") (pin "15") (pin "16") (pin "17") (pin "18") (pin "19") (pin "20") (pin "21") (pin "22") (pin "23") (pin "24") (pin "25") (pin "26") (pin "27") (pin "28") (pin "29") (pin "30") (pin "31") (pin "32") (pin "33") (pin "34") (pin "35") (pin "36") (pin "37") (pin "38") (pin "39") (pin "40") (pin "41") (pin "42") (pin "43") (pin "44") (pin "45") (pin "46") (pin "47") (pin "48") (instances (project "fasoguardian-v1" (path "/575af4e1-e15c-5e7c-a7b6-b5580dce1053/f00164bc-1320-5990-b001-d3d612522a42" (reference "U1") (unit 1)))))
 (global_label "3V3" (shape passive) (at 54.61 44.45 90) (fields_autoplaced yes) (effects (font (size 1.27 1.27)) (justify left)) (property "Intersheetrefs" "${INTERSHEET_REFS}" (at 54.61 44.45 0) (effects (font (size 1.27 1.27)) (hide yes))))
 (global_label "MCU_PWRKEY" (shape passive) (at 44.45 67.31 180) (fields_autoplaced yes) (effects (font (size 1.27 1.27)) (justify right)) (property "Intersheetrefs" "${INTERSHEET_REFS}" (at 44.45 67.31 0) (effects (font (size 1.27 1.27)) (hide yes))))
